File: UccMicroDuino/UccMicroDuino.kicad_sch (KiCad schematic)
At the start: 14 parts, among them J1 Pcb USB Type A, J2 Header, U1 ATtiny85-20SU

Commit message: Add files via upload
Actualización proyecto KiCad
Parts:
- D3: value 3.6v 1/2mW -> 3.6V 1/2mW
- D4: value Led Green -> LED Green
- D5: value Led Red -> LED Red
- R1: value 1.5KΩ 5% 1/8W -> 1.5KΩ 5% 1/8w
- R2, R3: value 68Ω 5% 1/8W -> 68Ω 5% 1/8W
Connections:
- net GND: now also R5.2; no longer R5.1
- net at D5.1 (K): now also R5.1; no longer R5.2
- net at D2.1 (K), J1.2 (D-), R1.2: now also R2.1; no longer R2.2
- net at J2.7 (Pin_7), U1.2 (XTAL1/PB3): now also R2.2; no longer R2.1
- net at J2.8 (Pin_8), U1.3 (XTAL2/PB4): now also R3.2; no longer R3.1
- net at D3.1 (K), J1.3 (D+): now also R3.1; no longer R3.2
Other:
- moved on the sheet: D5, U1
